Commit message: updated with second robot and ekf

File: install/my_robot_description/share/my_robot_description/urdf/robot_description.urdf.xacro (robot description, xacro)
@@ -189,5 +189,5 @@
         <parent link="base_link" />
         <child link="lidar" />
-        <origin xyz="0.15 0 0.0" rpy="0 0 0" />
+        <origin xyz="0.15 0 0.15" rpy="0 0 0" />
     </joint>
 </robot>

File: install/my_robot_description/share/my_robot_description/urdf/robot_description_gazebo.xacro (robot description, xacro)
@@ -42,5 +42,5 @@
     <plugin filename="libgazebo_ros_imu_sensor.so" name="imu_plugin">
         <ros>
-          <namespace>/demo</namespace>
+          <topicName>imu_data</topicName>
           <remapping>~/out:=imu</remapping>
         </ros>
